File: electronics/mainstep.sch (KiCad schematic (older format))
At the start: 51 parts, among them IC1 DRV8834_SOP, SW1 Reset, SW2 HWB, SW3 Summer Time, SW4 RST-RTC, U1 ATmega32U4-AU, U2 DS3231N, X1 CRYSTAL

Commit message: updated values
470R led drop resistors
Parts:
- R19, R20: value 500R -> 470R
Changed lines of the file:
@@
 LIBS:IP4220CZ6
 LIBS:mainstep-cache
-EELAYER 24 0
+EELAYER 27 0
 EELAYER END
 $Descr A4 11693 8268
@@
 Sheet 1 1
 Title "Mains Stepper Clock"
-Date "23 Jun 2014"
+Date "7 aug 2014"
 Rev ""
 Comp "VapourForge"
@@
 P 8100 950
 F 0 "R20" H 8030 1000 25  0000 C CNN
-F 1 "500R" H 8170 1000 20  0000 C CNN
+F 1 "470R" H 8170 1000 20  0000 C CNN
 F 2 "" H 8100 950 60  0000 C CNN
 F 3 "" H 8100 950 60  0000 C CNN
@@
 P 5700 6000
 F 0 "R19" H 5630 6050 25  0000 C CNN
-F 1 "500R" H 5770 6050 20  0000 C CNN
+F 1 "470R" H 5770 6050 20  0000 C CNN
 F 2 "" H 5700 6000 60  0000 C CNN
 F 3 "" H 5700 6000 60  0000 C CNN
