File: electronics/mainstep.kicad_pcb (KiCad board)
At the start: 2 copper layers, 100 x 50 mm, 56 parts, among them IC1 DRV8834_SOP, SW1 Reset, SW2 HWB, SW3 Summer Time, SW4 RST-RTC, U1 ATmega32U4-AU, U2 DS3231N, X1 CRYSTAL

Commit message: quit kicad
Parts:
- moved Usb_Gnd1 1.02 mm to (83.8, 85.1)
- moved VBus1 0.52 mm to (83.8, 90.8)
- moved D+1 0.13 mm to (83.8, 88.9)
- moved D-1 0.13 mm to (83.8, 87.0)
Connections:
- U1 pad 10: Net-(U1-Pad10) -> Net-(R12-Pad2)
Routing:
- net Net-(R12-Pad2): track 17.9 -> 83.8 mm, vias 0 -> 2
- net GND: track 385.6 -> 444.4 mm, vias 4 -> 6
- net +5V: track 308.8 -> 353.9 mm
- net Net-(U1-Pad10): track 8.34 -> 0.00 mm, vias 1 -> 0
Other:
- net class phat added: clearance 0.254, trace_width 2, via_dia 2.5, via_drill 1.2
- board text added: "Vapourforge.com RTC goverened USB Powered Stepper Driver Version 0.1 2014-07-14"
- board text removed: "1"
- board text removed: "Vapourforge.com RTC goverened USB Powered Stepper Driver Version 0.1 2014-07-08"
